File: Carte allumage/Shunt/command.kicad_sch (KiCad schematic)
At the start: 6 parts, among them U3 TLP3545AF, U4 TLP3545AF

Commit message: Pull-down signal on shunt
Parts:
- added R10: R, Resistor_SMD:R_0805_2012Metric_Pad1.20x1.40mm_HandSolder, symbol Device:R
Connections:
- net GND_SQ: now also R10.1
- net signal: now also R10.2

Commit message: test
Parts:
- added R11: R, Resistor_SMD:R_0805_2012Metric_Pad1.20x1.40mm_HandSolder, symbol Device:R
Connections:
- net GND_SQ: now also R11.1
- net signal: now also R11.2
