File: SUITON_telem/SUITON/SUITON.kicad_sch (KiCad schematic)
At the start: 0 parts

Commit message: Sensor
Other:
- added sheet Sensor (untitled.kicad_sch)
- added sheet Telem & Data (logging.kicad_sch)
Changed lines of the file:
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@@
+		)
+	)
+	(sheet
+		(at 86.36 30.48)
+		(size 54.61 29.21)
+		(fields_autoplaced yes)
+		(stroke
+			(width 0.1524)
+			(type solid)
+		)
+		(fill
+			(color 0 0 0 0.0000)
+		)
+		(property "Sheetname" "Telem & Data"
+			(at 86.36 29.7684 0)
+			(effects
+				(font
+					(size 1.27 1.27)
+				)
+				(justify left bottom)
+			)
+		)
+		(property "Sheetfile" "logging.kicad_sch"
+			(at 86.36 60.2746 0)
+			(effects
+				(font
+					(size 1.27 1.27)
+				)
+				(justify left top)
+			)
+		)
+		(instances
+			(project "SUITON"
+				(path "/2c712d4c-abcd-440d-8aed-9b8cbcb1a05a"
+					(page "4")
+				)
+			)
+		)
+	)
+	(sheet
+		(at 181.61 77.47)
+		(size 58.42 27.94)
+		(fields_autoplaced yes)
+		(stroke
+			(width 0.1524)
+			(type solid)
+		)
+		(fill
+			(color 0 0 0 0.0000)
+		)
+		(property "Sheetname" "Sensor"
+			(at 181.61 76.7584 0)
+			(effects
+				(font
+					(size 1.27 1.27)
+				)
+				(justify left bottom)
+			)
+		)
+		(property "Sheetfile" "untitled.kicad_sch"
+			(at 181.61 105.9946 0)
+			(effects
+				(font
+					(size 1.27 1.27)
+				)
+				(justify left top)
+			)
+		)
+		(instances
+			(project "SUITON"
+				(path "/2c712d4c-abcd-440d-8aed-9b8cbcb1a05a"
+					(page "3")
+				)
+			)
 		)
 	)

Commit message: power management
Other:
- added sheet Power (Power.kicad_sch)
- company: (none) -> S.T.A.R.
- title: (none) -> SUITON PRO
Changed lines of the file:
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@@
 	(generator_version "8.0")
 	(paper "A4")
+	(title_block
+		(title "SUITON PRO")
+		(date "2026-10-01")
+		(company "S.T.A.R.")
+		(comment 1 "Axel BOULAROT")
+		(comment 2 "Versatile Flight Controller for rocket and more")
+	)
+	(sheet
+		(at 86.36 74.93)
+		(size 53.34 30.48)
+		(fields_autoplaced yes)
+		(stroke
+			(width 0.1524)
+			(type solid)
+		)
+		(fill
+			(color 0 0 0 0.0000)
+		)
+		(property "Sheetname" "Power"
+			(at 86.36 74.2184 0)
+			(effects
+				(font
+					(size 1.27 1.27)
+				)
+				(justify left bottom)
+			)
+		)
+		(property "Sheetfile" "Power.kicad_sch"
+			(at 86.36 105.9946 0)
+			(effects
+				(font
+					(size 1.27 1.27)
+				)
+				(justify left top)
+			)
+		)
+		(instances
+			(project "SUITON"
+				(path "/2c712d4c-abcd-440d-8aed-9b8cbcb1a05a"
+					(page "5")
+				)
+			)
+		)
+	)
 	(sheet
 		(at 181.61 30.48)

Commit message: SUITON PRO
Other:
- added sheet COM (com.kicad_sch)
Changed lines of the file:
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@@
 			(project "SUITON"
 				(path "/2c712d4c-abcd-440d-8aed-9b8cbcb1a05a"
-					(page "5")
+					(page "2")
 				)
 			)
@@
 			(project "SUITON"
 				(path "/2c712d4c-abcd-440d-8aed-9b8cbcb1a05a"
-					(page "2")
+					(page "3")
 				)
 			)
@@
 			(project "SUITON"
 				(path "/2c712d4c-abcd-440d-8aed-9b8cbcb1a05a"
-					(page "4")
+					(page "5")
 				)
 			)
@@
 			(project "SUITON"
 				(path "/2c712d4c-abcd-440d-8aed-9b8cbcb1a05a"
-					(page "3")
+					(page "4")
 				)
 			)
+		)
+	)
+	(sheet
+		(at 181.61 124.46)
+		(size 58.42 29.21)
+		(fields_autoplaced yes)
+		(stroke
+			(width 0.1524)
+			(type solid)
+		)
+		(fill
+			(color 0 0 0 0.0000)
+		)
+		(property "Sheetname" "COM"
+			(at 181.61 123.7484 0)
+			(effects
+				(font
+					(size 1.27 1.27)
+				)
+				(justify left bottom)
+			)
+		)
+		(property "Sheetfile" "com.kicad_sch"
+			(at 181.61 154.2546 0)
+			(effects
+				(font
+					(size 1.27 1.27)
+				)
+				(justify left top)
+			)
+		)
+		(instances
+			(project "SUITON"
+				(path "/2c712d4c-abcd-440d-8aed-9b8cbcb1a05a"
+					(page "6")
+				)
+			)
