File: SUITON_telem/SUITON/mcu.kicad_sch (KiCad schematic)
At the start: 22 parts, among them U1 STM32H523ZCT6

Commit message: Flash mode
Parts:
- added C21, C22: 12pF, Capacitor_SMD:C_0603_1608Metric, symbol Device:C
- added C23, C24: 100nF, Capacitor_SMD:C_0603_1608Metric, symbol Device:C
- added J1: USB_C_Receptacle_USB2.0_14P, symbol Connector:USB_C_Receptacle_USB2.0_14P
- added R2: 47 Ω, symbol Device:R
- added R3, R4: 5.1kΩ, symbol Device:R
- added S1, S2: B3U-1000P, B3U-1000P:SW_B3U-1000P, symbol B3U-1000P:B3U-1000P
- added X1: ABM3B-8.000MHZ-10-1UT, XTAL4P_ABM3B_ABR, symbol 2026-09-29_10-16-59:ABM3B-8.000MHZ-10-1UT
Connections:
- net +3V3: now also S2.1
- net GND: now also C21.2, C22.2, C23.2, C24.2, J1.A1 (GND), J1.A12 (GND), J1.B1 (GND), J1.B12 (GND), J1.S1 (SHIELD), R2.2, R3.2, R4.2, S1.1, X1.2, X1.4
- net BOOT: now reaches U1.138 (BOOT0)
- net BOOT: now also C24.1, R2.1, S2.2
- net OSC_IN: now reaches U1.23 (PH0-OSC_IN)
- net OSC_IN: now also C22.1, X1.1
- net OSC_OUT: now reaches U1.24 (PH1-OSC_OUT)
- net OSC_OUT: now also C21.1, X1.3
- net NRST: now reaches U1.25 (NRST)
- net NRST: now also C23.1, S1.2
- net USB_DM: now reaches U1.103 (PA11)
- net USB_DM: now also J1.A7 (D-), J1.B7 (D-)
- net USB_DP: now reaches U1.104 (PA12)
- net USB_DP: now also J1.A6 (D+), J1.B6 (D+)
- net SWDIO: now reaches U1.105 (PA13)
- net SWCLK: now reaches U1.109 (PA14)
- net SWO: now reaches U1.133 (PB3)
- new net: J1.B5 (CC2), R4.1
- new net: J1.A5 (CC1), R3.1
- new net +5V_USB: J1.A4 (VBUS), J1.A9 (VBUS), J1.B4 (VBUS), J1.B9 (VBUS)
- no-connect marks 0 -> 2
Other:
- moved on the sheet: C1, C10, C11, C12, C13, C14, C15, C16, C17, C18, C19, C2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

Commit message: Sensor
Parts:
- added J2: Conn_01x06_Pin, symbol Connector:Conn_01x06_Pin
Connections:
- net +3V3: now also J2.1 (Pin_1)
- net GND: now also J2.3 (Pin_3)
- net NRST: now also J2.5 (Pin_5)
- net SWCLK: now also J2.2 (Pin_2)
- net SWDIO: now also J2.4 (Pin_4)
- net SWO: now also J2.6 (Pin_6)
- net UART1_TX: now reaches U1.101 (PA9)
- net UART1_RX: now reaches U1.102 (PA10)
- net SPI1_NSS: now reaches U1.40 (PA4)
- net SPI1_SCK: now reaches U1.41 (PA5)
- net SPI1_MISO: now reaches U1.42 (PA6)
- net SPI1_MOSI: now reaches U1.43 (PA7)
- no-connect marks 2 -> 4

Commit message: power management
Connections:
- net OCTOSPI1_NCS: now reaches U1.136 (PB6)
- net OCTOSPI1_IO1: now reaches U1.46 (PB0)
- net OCTOSPI1_IO0: now reaches U1.47 (PB1)
- net OCTOSPI1_CLK: now reaches U1.48 (PB2)
- net SPI1_MISO renamed OCTOSPI1_IO3
- net SPI1_MOSI renamed OCTOSPI1_IO2
- net SPI1_NSS: no longer names the net of U1.40 (PA4)
- net SPI1_SCK: no longer names the net of U1.41 (PA5)
Other:
- company: (none) -> S.T.A.R.
- title: (none) -> SUITON PRO
Changed lines of the file:
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@@
 	(generator_version "8.0")
 	(paper "A3")
+	(title_block
+		(title "SUITON PRO")
+		(date "2026-10-01")
+		(company "S.T.A.R.")
+		(comment 1 "Axel BOULAROT")
+		(comment 2 "Versatile Flight Controller for rocket and more")
+	)
 	(junction
 		(at 304.8 168.91)
@@
 		)
 	)
-	(global_label "SPI1_MOSI"
+	(global_label "OCTOSPI1_IO1"
 		(shape input)
-		(at 111.76 64.77 180)
+		(at 111.76 90.17 180)
 		(fields_autoplaced yes)
 		(effects
@@
 		)
 		(property "Intersheetrefs" "${INTERSHEET_REFS}"
-			(at 98.9172 64.77 0)
+			(at 95.47 90.17 0)
 			(effects
 				(font
@@
 		)
 	)
-	(global_label "SPI1_SCK"
+	(global_label "OCTOSPI1_CLK"
 		(shape input)
-		(at 111.76 59.69 180)
+		(at 111.76 95.25 180)
 		(fields_autoplaced yes)
 		(effects
@@
 		)
 		(property "Intersheetrefs" "${INTERSHEET_REFS}"
-			(at 99.7639 59.69 0)
+			(at 95.0467 95.25 0)
 			(effects
 				(font
@@
 		)
 	)
-	(global_label "SPI1_MISO"
+	(global_label "OCTOSPI1_IO3"
 		(shape input)
 		(at 111.76 62.23 180)
@@
 		)
 		(property "Intersheetrefs" "${INTERSHEET_REFS}"
-			(at 98.9172 62.23 0)
+			(at 95.47 62.23 0)
 			(effects
 				(font
@@
 		)
 	)
-	(global_label "SPI1_NSS"
+	(global_label "OCTOSPI1_IO0"
 		(shape input)
-		(at 111.76 57.15 180)
+		(at 111.76 92.71 180)
 		(fields_autoplaced yes)
 		(effects
@@
 		)
 		(property "Intersheetrefs" "${INTERSHEET_REFS}"
-			(at 99.7639 57.15 0)
+			(at 95.47 92.71 0)
 			(effects
 				(font
+					(size 1.27 1.27)
+				)
+				(justify right)
+				(hide yes)
+			)
+		)
+	)
+	(global_label "OCTOSPI1_IO2"
+		(shape input)
+		(at 111.76 64.77 180)
+		(fields_autoplaced yes)
+		(effects
+			(font
+				(size 1.27 1.27)
+			)
+			(justify right)
+		)
+		(property "Intersheetrefs" "${INTERSHEET_REFS}"
+			(at 95.47 64.77 0)
+			(effects
+				(font
+					(size 1.27 1.27)
+				)
+				(justify right)
+				(hide yes)
+			)
+		)
+	)
+	(global_label "OCTOSPI1_NCS"
+		(shape input)
+		(at 111.76 105.41 180)
+		(fields_autoplaced yes)
+		(effects
+			(font
+				(size 1.27 1.27)
+			)
+			(justify right)
+		)
+		(property "Intersheetrefs" "${INTERSHEET_REFS}"
+			(at 94.8048 105.41 0)
+			(effects
+				(font

Commit message: SUITON PRO
Connections:
- net UART1_RX: now also U1.35 (PA1); no longer U1.102 (PA10)
- net UART1_TX: now also U1.34 (PA0); no longer U1.101 (PA9)
- net INT1_IMU1: now reaches U1.1 (PE2)
- net RESET_RF: now reaches U1.10 (PF0)
- net DIO5_RF: now reaches U1.11 (PF1)
- net DIO3_RF: now reaches U1.12 (PF2)
- net GPIO10: now reaches U1.124 (PG9)
- net GPIO11: now reaches U1.125 (PG10)
- net GPIO12: now reaches U1.126 (PG11)
- net GPIO13: now reaches U1.127 (PG12)
- net GPIO14: now reaches U1.128 (PG13)
- net GPIO15: now reaches U1.129 (PG14)
- net DIO4_RF: now reaches U1.13 (PF3)
- net GPIO16: now reaches U1.132 (PG15)
- net DIO0_RF: now reaches U1.14 (PF4)
- net INT_BMP: now reaches U1.141 (PE0)
- net DIO1_RF: now reaches U1.15 (PF5)
- net DIO2_RF: now reaches U1.18 (PF6)
- net BUTTON1_OUT: now reaches U1.19 (PF7)
- net INT2_IMU1: now reaches U1.2 (PE3)
- net BUTTON2_OUT: now reaches U1.20 (PF8)
- net GPIO19: now reaches U1.21 (PF9)
- net GPIO20: now reaches U1.22 (PF10)
- net INT1_IMU2: now reaches U1.3 (PE4)
- net INT2_IMU2: now reaches U1.4 (PE5)
- net ADC5: now reaches U1.49 (PF11)
- net EXTINT_SAM: now reaches U1.5 (PE6)
- net ADC6: now reaches U1.50 (PF12)
- net ADC7: now reaches U1.53 (PF13)
- net ADC8: now reaches U1.54 (PF14)
- net GPIO21: now reaches U1.55 (PF15)
- net GPIO1: now reaches U1.56 (PG0)
- net GPIO2: now reaches U1.57 (PG1)
- net RESET_SAM: now reaches U1.58 (PE7)
- net SAFEBOOT_SAM: now reaches U1.59 (PE8)
- net TIMEPULSE_SAM: now reaches U1.63 (PE10)
- net SCLK_SPI3: now reaches U1.65 (PE12)
- net MISO_SPI3: now reaches U1.66 (PE13)
- net MOSI_SPI3: now reaches U1.67 (PE14)
- net GPIO3: now reaches U1.87 (PG2)
- net GPIO4: now reaches U1.88 (PG3)
- net GPIO5: now reaches U1.89 (PG4)
- net GPIO6: now reaches U1.90 (PG5)
- net GPIO7: now reaches U1.91 (PG6)
- net GPIO8: now reaches U1.92 (PG7)
- net GPIO9: now reaches U1.93 (PG8)
- net SCLK_SPI2: now reaches U1.111 (PC10)
- net MISO_SPI2: now reaches U1.112 (PC11)
- net MOSI_SPI2: now reaches U1.113 (PC12)
- net CS_IMU1: now reaches U1.114 (PD0)
- net CS_IMU2: now reaches U1.115 (PD1)
- net CS_BMP: now reaches U1.116 (PD2)
- net CS_MMC: now reaches U1.117 (PD3)
- net CS_SD: now reaches U1.118 (PD4)
- net CS_RF: now reaches U1.119 (PD5)
- net SCL_I2C3: now reaches U1.122 (PD6)
- net SDA_I2C3: now reaches U1.123 (PD7)
- net SCL_I2C1: now reaches U1.139 (PB8)
- net SDA_I2C1: now reaches U1.140 (PB9)
- net ADC1: now reaches U1.26 (PC0)
- net ADC2: now reaches U1.27 (PC1)
- net ADC3: now reaches U1.28 (PC2)
- net ADC4: now reaches U1.29 (PC3)
- net SCL_I2C2: now reaches U1.69 (PB10)
- net SDA_I2C2: now reaches U1.73 (PB12)
- net SCLK_SPI1: now reaches U1.74 (PB13)
- net MISO_SPI1: now reaches U1.75 (PB14)
- net MOSI_SPI1: now reaches U1.76 (PB15)
- net PWM1: now reaches U1.81 (PD12)
- net BUZZER: now reaches U1.82 (PD13)
- net PWM3: now reaches U1.85 (PD14)
- net PWM4: now reaches U1.86 (PD15)
- net PWM5: now reaches U1.96 (PC6)
- net PWM6: now reaches U1.97 (PC7)
- net PWM7: now reaches U1.98 (PC8)
- net PWM8: now reaches U1.99 (PC9)
- new net UART2_RX: U1.102 (PA10)
- new net UART2_TX: U1.101 (PA9)
Other:
- note added: "MCU & IHM"
- moved on the sheet: C1, C10, C11, C12, C13, C14, C15, C16, C17, C18, C19, C2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
