File: SUITON_telem/SUITON_mini/power.kicad_sch (KiCad schematic)
At the start: 33 parts, among them J1 Conn_01x02_Pin, Q1 2N7002, Q2 AO3407A, U2 TPS63070RNMR, U3 TPS2121RUXR, U4 AP2112K-3.3TRG1

Commit message: New rf module
Parts:
- removed Q1: 2N7002, Package_TO_SOT_SMD:SOT-23, symbol Transistor_FET:2N7002
- added Q5: BSS138, Package_TO_SOT_SMD:SOT-23, symbol Transistor_FET:BSS138
Connections:
- net GND: now also Q5.2 (S)
- net at R4.1, U2.1 (PS/SYNC), U2.14 (EN): now also Q5.3 (D)
- net at R1.2, R2.2: now also Q5.1 (G)
