File: SUITON_telem/SUITON_mini/_autosave-power.kicad_sch (KiCad schematic)
At the start: 32 parts, among them J1 Conn_01x02_Pin, Q2 AO3407A, Q5 BSS138, U2 TPS63070RNMR, U3 TPS2121RUXR, U4 AP2112K-3.3TRG1

Commit message: Commencement du placement des composants
Parts:
- C4: footprint Capacitor_SMD:C_0402_1005Metric -> Resistor_SMD:R_0402_1005Metric
- C9: footprint Capacitor_SMD:C_0603_1608Metric -> Resistor_SMD:R_0201_0603Metric
- R10, R11, R12, R8, R9: footprint (none) -> Resistor_SMD:R_0201_0603Metric
- R2: value 100kΩ -> 10kΩ
Changed lines of the file:
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@@
 			)
 		)
-		(property "Footprint" ""
+		(property "Footprint" "Resistor_SMD:R_0201_0603Metric"
 			(at 177.038 87.63 90)
 			(hide yes)
@@
 			)
 		)
-		(property "Value" "100kΩ"
+		(property "Value" "10kΩ"
 			(at 46.228 81.026 0)
 			(show_name no)
@@
 			)
 		)
-		(property "Footprint" ""
+		(property "Footprint" "Resistor_SMD:R_0201_0603Metric"
 			(at 156.972 74.93 90)
 			(hide yes)
@@
 			)
 		)
-		(property "Footprint" "Capacitor_SMD:C_0402_1005Metric"
+		(property "Footprint" "Resistor_SMD:R_0402_1005Metric"
 			(at 116.5352 81.28 0)
 			(hide yes)
@@
 			)
 		)
-		(property "Footprint" ""
+		(property "Footprint" "Resistor_SMD:R_0201_0603Metric"
 			(at 166.37 76.962 90)
 			(hide yes)
@@
 			)
 		)
-		(property "Footprint" ""
+		(property "Footprint" "Resistor_SMD:R_0201_0603Metric"
 			(at 177.038 72.39 90)
 			(hide yes)
@@
 			)
 		)
-		(property "Footprint" ""
+		(property "Footprint" "Resistor_SMD:R_0201_0603Metric"
 			(at 162.56 66.802 90)
 			(hide yes)
@@
 			)
 		)
-		(property "Footprint" "Capacitor_SMD:C_0603_1608Metric"
+		(property "Footprint" "Resistor_SMD:R_0201_0603Metric"
 			(at 164.7952 91.44 0)
 			(hide yes)
