File: SUITON_telem/SUITON_mini/sensor.kicad_sch (KiCad schematic)
At the start: 17 parts, among them U10 LSM6DSV320XTR, U6 MMC5983MA, U7 ISM330DHCXTR, U8 SAM-M10Q-00B, U9 BMP581

Commit message: New rf module
Parts:
- removed C12: 1uF, Capacitor_SMD:C_0603_1608Metric, symbol Device:C
- removed C15: 10uF, Capacitor_SMD:C_0603_1608Metric, symbol Device:C
- removed U6: MMC5983MA, MMC5983MA_MEM, symbol 2026-09-30_16-50-22:MMC5983MA
Connections:
- no-connect marks 11 -> 5
Other:
- note removed: "MAGNETOMETER"

Commit message: Premier placement global
Parts:
- removed R14, R15: 0Ω, symbol Device:R
- removed R16, R17: 10Ω, symbol Device:R
- C13, C14, C16, C17, C18, C19: footprint Capacitor_SMD:C_0603_1608Metric -> Capacitor_SMD:C_0402_1005Metric
Connections:
- net +3V3: now also C16.2, C18.1, U9.1 (VDDIO), U9.10 (VDD)
- no-connect marks 5 -> 7
