File: SUITON_telem/SUITON_mini/ihm_pyro.kicad_sch (KiCad schematic)
At the start: 21 parts, among them Q2 BSS138, U11 74HC2G14GW_125

Commit message: SUITON mini
Parts:
- removed C48, C49, C50, C53: 100nF, Capacitor_SMD:C_0603_1608Metric, symbol Device:C
- removed C51, C52: 1uF, Capacitor_SMD:C_0603_1608Metric, symbol Device:C
- removed D5: WS2812B, LED_SMD:LED_WS2812B_PLCC4_5.0x5.0mm_P3.2mm, symbol LED:WS2812B
- removed D7: 1N4148, Diode_SMD:D_0603_1608Metric, symbol Diode:1N4148
- removed Q2: BSS138, Package_TO_SOT_SMD:SOT-23, symbol Transistor_FET:BSS138
- removed R26, R27, R28, R29, R30: 10kΩ, symbol Device:R
- removed R31: 1kΩ, symbol Device:R
- removed S3, S4: B3U-1000P, B3U-1000P:SW_B3U-1000P, symbol B3U-1000P:B3U-1000P
- added C20, C21, C27: 100nF, Capacitor_SMD:C_0603_1608Metric, symbol Device:C
- added C25, C26: 1uF, Capacitor_SMD:C_0603_1608Metric, symbol Device:C
- added D5: 1N4148, Diode_SMD:D_0603_1608Metric, symbol Diode:1N4148
- added Q3: BSS138, Package_TO_SOT_SMD:SOT-23, symbol Transistor_FET:BSS138
- added R18: 1kΩ, symbol Device:R
- added R19, R20, R21, R22, R23: 10kΩ, symbol Device:R
- added S1: B3U-1000P, B3U-1000P:SW_B3U-1000P, symbol B3U-1000P:B3U-1000P
- added TP1: Jack, symbol Connector:TestPoint
Connections:
- net +3V3: now also C27.2, R20.2, R21.1
- net +5V: now also C20.2, C21.2, D5.1 (K)
- net BUZZER: now also R18.1
- net GND: now also C20.1, C21.1, C25.1, C26.1, C27.1, Q3.2 (S), R19.1, S1.1
- net at LS1.N: now also D5.2 (A), Q3.3 (D)
- net at U11.1 (1A): now also R22.2
- net at U11.3 (2A): now also R23.1
- net at D6.4 (DIN): now also D4.2 (DOUT)
- new net: C26.2, R21.2, R23.2, TP1.1
- new net: Q3.1 (G), R18.2, R19.2
- new net: C25.2, R20.1, R22.1, S1.2
Other:
- title: SUITON PRO -> SUITON mini

Commit message: New rf module
Parts:
- removed C25, C26: 1uF, Capacitor_SMD:C_0603_1608Metric, symbol Device:C
- removed C27: 100nF, Capacitor_SMD:C_0603_1608Metric, symbol Device:C
- removed R20, R21, R22, R23: 10kΩ, symbol Device:R
- removed S1: B3U-1000P, B3U-1000P:SW_B3U-1000P, symbol B3U-1000P:B3U-1000P
- removed TP1: Jack, symbol Connector:TestPoint
- removed U11: 74HC2G14GW_125, TSSOP6_SOT363-2_NEX, symbol 2026-10-04_17-37-41:74HC2G14GW_125
Other:
- note removed: "BUTTON ON SCHMITT TRIGGER"
- moved on the sheet: C20, C21, D4, D5, D6, LS1, Q3, R18, R19

Commit message: Premier placement global
Parts:
- removed R18: 1kΩ, symbol Device:R
- R19: footprint (none) -> Resistor_SMD:R_0603_1608Metric
Connections:
- net BUZZER: now also Q3.1 (G), R19.2
Changed lines of the file:
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@@
 	(wire
 		(pts
-			(xy 193.04 92.71) (xy 190.5 92.71)
+			(xy 190.5 92.71) (xy 203.2 92.71)
 		)
 		(stroke
@@
 		(pts
 			(xy 199.39 74.93) (xy 210.82 74.93)
-		)
-		(stroke
-			(width 0)
-			(type default)
-		)
-	)
-	(wire
-		(pts
-			(xy 200.66 92.71) (xy 203.2 92.71)
 		)
 		(stroke
@@
 			)
 		)
-		(property "Footprint" ""
+		(property "Footprint" "Resistor_SMD:R_0603_1608Metric"
 			(at 204.978 96.52 90)
 			(hide yes)
@@
 					(unit 1)
 				)
-			)
-		)
-	)
-	(symbol
-		(lib_id "Device:R")
-		(at 196.85 92.71 90)
-		(unit 1)
-		(body_style 1)
-		(exclude_from_sim no)
-		(in_bom yes)
-		(on_board yes)
-		(in_pos_files yes)
-		(dnp no)
-		(property "Reference" "R18"
-			(at 197.104 88.392 90)
-			(show_name no)
-			(do_not_autoplace no)
-			(effects
-				(font
-					(size 1.27 1.27)
-				)
-			)
-		)
-		(property "Value" "1kΩ"
-			(at 196.85 90.424 90)
-			(show_name no)
-			(do_not_autoplace no)
-			(effects
-				(font
-					(size 1.27 1.27)
-				)
-			)
-		)
-		(property "Footprint" ""
-			(at 196.85 94.488 90)
-			(hide yes)
-			(show_name no)
-			(do_not_autoplace no)
-			(effects
-				(font
-					(size 1.27 1.27)
-				)
-			)
-		)
-		(property "Datasheet" ""
-			(at 196.85 92.71 0)
-			(hide yes)
-			(show_name no)
-			(do_not_autoplace no)
-			(effects
-				(font
-					(size 1.27 1.27)
-				)
-			)
-		)
-		(property "Description" "Resistor"
-			(at 196.85 92.71 0)
-			(hide yes)
-			(show_name no)
-			(do_not_autoplace no)
-			(effects
-				(font
-					(size 1.27 1.27)
-				)
-			)
-		)
-		(pin "2"
-		)
-		(pin "1"
-		)
-		(instances
-			(project "SUITON_mini"
-				(path "/651dea4f-1e55-4052-accd-e9842c395f76/873eb0e4-6ac7-40ec-9166-17753800617b"
-					(reference "R18")
-					(unit 1)
-				)

Commit message: Shape
Parts:
- removed C21: 100nF, Capacitor_SMD:C_0603_1608Metric, symbol Device:C
- removed D6: WS2812B, LED_SMD:LED_WS2812B_PLCC4_5.0x5.0mm_P3.2mm, symbol LED:WS2812B
- added H1, H2, H3, H4: MountingHole_Pad, MountingHole:MountingHole_2.2mm_M2_Pad_Via, symbol Mechanical:MountingHole_Pad
Connections:
- net GND: now also H1.1, H2.1, H3.1, H4.1
Other:
- moved on the sheet: C20, D4
