File: SUITON_telem/SUITON_mini/memory.kicad_sch (KiCad schematic)
At the start: 7 parts, among them IC1 W25Q128JVEIM, J3 CON-SMA-EDGE-S, U1 RFM95W-868S2

Commit message: New rf module
Parts:
- removed J3: CON-SMA-EDGE-S, CON-SMA-EDGE-S:RFSOLUTIONS_CON-SMA-EDGE-S, symbol CON-SMA-EDGE-S:CON-SMA-EDGE-S
- removed U1: RFM95W-868S2, RFM95W-868S2:XCVR_RFM95W-868S2, symbol RFM95W-868S2:RFM95W-868S2
- added AE1: Antenna_Shield, Footprints:SMA_EdgeMount, symbol Device:Antenna_Shield
- added C12: 100n, Capacitor_SMD:C_0402_1005Metric, symbol Device:C_Small
- added C24: 100nF, Capacitor_SMD:C_0603_1608Metric, symbol Device:C
- added C25: 10uF, Capacitor_SMD:C_0603_1608Metric, symbol Device:C
- added L2: 330n, Inductor_SMD:L_0402_1005Metric, symbol Device:L_Small
- added Q4: BSS138, Package_TO_SOT_SMD:SOT-23, symbol Transistor_FET:BSS138
- added R20: 100k, Resistor_SMD:R_0402_1005Metric, symbol Device:R
- added R21, R22: 10k, Resistor_SMD:R_0402_1005Metric, symbol Device:R
- added U6: E22-900MM22S, E22-900MM22S_BYT, symbol 2026-10-06_06-26-22:E22-900MM22S
Connections:
- net +3V3: now also C24.2, C25.2, U6.1 (VCC)
- net ANT: now also AE1.1 (A), L2.1, U6.6 (ANT)
- net CS_RF: now also U6.14 (NSS)
- net DIO1_RF: now also U6.20 (DIO1)
- net GND: now also AE1.2 (Shield), C12.2, C24.1, C25.1, L2.2, Q4.2 (S), R22.1, U6.16 (GND), U6.2 (GND), U6.7 (GND)
- net MISO_SPI2: now also U6.12 (MISO)
- net MOSI_SPI2: now also U6.13 (MOSI)
- net RESET_RF: now also C12.1, R20.2, U6.3 (NRST)
- net SCK_SPI2: now also U6.15 (SCK)
- new net +3.3V: R20.1, R21.1
- new net BUSY_RF: U6.11 (BUSY)
- new net RX_EN: Q4.3 (D), R21.2, U6.10 (RXEN)
- new net TX_EN: Q4.1 (G), R22.2, U6.19 (DIO2), U6.9 (TXEN)
- no-connect marks 3 -> 2
Other:
- moved on the sheet: C22, C23, IC1, R30, R31

Commit message: Premier placement global
Parts:
- removed IC1: W25Q128JVEIM, SON127P800X600X80-9N-D, symbol W25Q128JVEIM:W25Q128JVEIM
- added U1: W25Q128JVPIQ, W25Q128JVPIQ:W25Q128JVPIQ, symbol W25Q128JVPIQ:W25Q128JVPIQ
- C22: footprint Capacitor_SMD:C_0603_1608Metric -> Capacitor_SMD:C_0402_1005Metric
- R30, R31: footprint (none) -> Resistor_SMD:R_0402_1005Metric
Connections:
- net +3V3: now also U1.8 (VCC); no longer C24.2, C25.2, U6.1 (VCC)
- net CS_MEM: now also U1.1 (CS)
- net GND: now also U1.4 (GND), U1.9 (GND)
- net MISO_SPI2: now also U1.2 (DO(IO1))
- net MOSI_SPI2: now also U1.5 (DI(IO0))
- net SCLK_SPI2: now also U1.6 (CLK)
- net at R30.2: now also U1.3 (/WP(IO2))
- net at R31.2: now also U1.7 (HOLD/RESET(IO3))
- new net +3V3_radio: C24.2, C25.2, U6.1 (VCC)
- no-connect marks 2 -> 1
Other:
- moved on the sheet: R30, R31

Commit message: Shape
Parts:
- removed AE1: Antenna_Shield, Footprints:SMA_EdgeMount, symbol Device:Antenna_Shield
- added E1: ANT-868-JJB-RA, ANT-868-JJB-RA:XDCR_ANT-868-JJB-RA, symbol ANT-868-JJB-RA:ANT-868-JJB-RA
Connections:
- net ANT: now also E1.1
Changed lines of the file:
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@@
+	)
+	(junction
+		(at 147.32 87.63)
+		(diameter 0)
+		(color 0 0 0 0)
 	)
 	(junction
@@
 	)
 	(junction
-		(at 147.32 87.63)
-		(diameter 0)
-		(color 0 0 0 0)
-	)
-	(junction
-		(at 36.83 64.77)
-		(diameter 0)
-		(color 0 0 0 0)
-	)
-	(junction
 		(at 93.98 102.87)
 		(diameter 0)
@@
 	(wire
 		(pts
+			(xy 36.83 78.74) (xy 36.83 72.39)
+		)
+		(stroke
+			(width 0)
+			(type default)
+		)
+	)
+	(wire
+		(pts
 			(xy 213.36 110.49) (xy 219.71 110.49)
 		)
@@
 	(wire
 		(pts
-			(xy 34.29 64.77) (xy 36.83 64.77)
-		)
-		(stroke
-			(width 0)
-			(type default)
-		)
-	)
-	(wire
-		(pts
 			(xy 139.7 87.63) (xy 139.7 86.36)
-		)
-		(stroke
-			(width 0)
-			(type default)
-		)
-	)
-	(wire
-		(pts
-			(xy 34.29 72.39) (xy 34.29 64.77)
 		)
 		(stroke
@@
 	)
 	(symbol
+		(lib_id "ANT-868-JJB-RA:ANT-868-JJB-RA")
+		(at 36.83 83.82 180)
+		(unit 1)
+		(body_style 1)
+		(exclude_from_sim no)
+		(in_bom yes)
+		(on_board yes)
+		(in_pos_files yes)
+		(dnp no)
+		(fields_autoplaced yes)
+		(property "Reference" "E1"
+			(at 40.64 84.0104 0)
+			(show_name no)
+			(do_not_autoplace no)
+			(effects
+				(font
+					(size 1.27 1.27)
+				)
+				(justify right)
+			)
+		)
+		(property "Value" "ANT-868-JJB-RA"
+			(at 40.64 86.5504 0)
+			(show_name no)
+			(do_not_autoplace no)
+			(effects
+				(font
+					(size 1.27 1.27)
+				)
+				(justify right)
+			)
+		)
+		(property "Footprint" "ANT-868-JJB-RA:XDCR_ANT-868-JJB-RA"
+			(at 36.83 83.82 0)
+			(hide yes)
+			(show_name no)
+			(do_not_autoplace no)
+			(effects
+				(font
+					(size 1.27 1.27)
+				)
+				(justify bottom)
+			)
+		)
+		(property "Datasheet" ""
+			(at 36.83 83.82 0)
+			(hide yes)
+			(show_name no)
+			(do_not_autoplace no)
+			(effects
+				(font
+					(size 1.27 1.27)
+				)
+			)
+		)
+		(property "Description" "868 MHz Right Angle Monopole Dome Antenna"
+			(at 36.83 83.82 0)
+			(hide yes)
+			(show_name no)
+			(do_not_autoplace no)
+			(effects
+				(font
+					(size 1.27 1.27)
+				)
+				(justify bottom)
+			)
+		)
+		(property "MF" "Linx Technologies"
+			(at 36.83 83.82 0)
+			(hide yes)
+			(show_name no)
+			(do_not_autoplace no)
+			(effects
+				(font
+					(size 1.27 1.27)
+				)
+				(justify bottom)
+			)
+		)
+		(property "MAXIMUM_PACKAGE_HEIGHT" "7 mm"
+			(at 36.83 83.82 0)
+			(hide yes)
+			(show_name no)
+			(do_not_autoplace no)
+			(effects
+				(font
+					(size 1.27 1.27)
+				)
+				(justify bottom)
+			)
+		)
+		(property "Package" "None"
+			(at 36.83 83.82 0)
+			(hide yes)
+			(show_name no)
+			(do_not_autoplace no)
+			(effects
+				(font
+					(size 1.27 1.27)
+				)
+				(justify bottom)
+			)
+		)
+		(property "Price" "None"
+			(at 36.83 83.82 0)
+			(hide yes)
+			(show_name no)
+			(do_not_autoplace no)
+			(effects
+				(font
+					(size 1.27 1.27)
+				)
+				(justify bottom)
+			)
+		)
+		(property "Check_prices" "https://www.snapeda.com/parts/ANT-868-JJB-RA/TE+Connectivity/view-part/?ref=eda"
+			(at 36.83 83.82 0)
+			(hide yes)
+			(show_name no)
+			(do_not_autoplace no)
+			(effects
+				(font
+					(size 1.27 1.27)
+				)
+				(justify bottom)
+			)
+		)
+		(property "STANDARD" "Manufacturer Recommendations"
+			(at 36.83 83.82 0)
+			(hide yes)
+			(show_name no)
+			(do_not_autoplace no)
+			(effects
+				(font
+					(size 1.27 1.27)
+				)
+				(justify bottom)
+			)
+		)
+		(property "PARTREV" "4/11/16"
+			(at 36.83 83.82 0)
+			(hide yes)
+			(show_name no)
+			(do_not_autoplace no)
+			(effects
+				(font
+					(size 1.27 1.27)
+				)
+				(justify bottom)
+			)
+		)
+		(property "SnapEDA_Link" "https://www.snapeda.com/parts/ANT-868-JJB-RA/TE+Connectivity/view-part/?ref=snap"
+			(at 36.83 83.82 0)
+			(hide yes)
+			(show_name no)
+			(do_not_autoplace no)
+			(effects
+				(font
+					(size 1.27 1.27)
+				)
+				(justify bottom)
+			)
+		)
+		(property "MP" "ANT-868-JJB-RA"
+			(at 36.83 83.82 0)
+			(hide yes)
+			(show_name no)
+			(do_not_autoplace no)
+			(effects
+				(font
+					(size 1.27 1.27)
+				)
+				(justify bottom)
+			)
+		)
+		(property "Availability" "In Stock"
+			(at 36.83 83.82 0)
+			(hide yes)
+			(show_name no)
+			(do_not_autoplace no)
+			(effects
+				(font
+					(size 1.27 1.27)
+				)
+				(justify bottom)
+			)
+		)
+		(property "MANUFACTURER" "Linx"
+			(at 36.83 83.82 0)
+			(hide yes)
+			(show_name no)
+			(do_not_autoplace no)
+			(effects
+				(font
+					(size 1.27 1.27)
+				)
+				(justify bottom)
+			)
+		)
+		(pin "1"
+		)
+		(instances
+			(project "SUITON_mini"
+				(path "/651dea4f-1e55-4052-accd-e9842c395f76/cbc1e4b3-87c3-4a09-a481-980e2b628052"
+					(reference "E1")
+					(unit 1)
+				)
+			)
+		)
+	)
+	(symbol
 		(lib_id "power:+3V3")
 		(at 177.8 78.74 90)
@@
 					(unit 1)
 				)
-			)
-		)
-	)
-	(symbol
-		(lib_id "Device:Antenna_Shield")
-		(at 36.83 77.47 180)
-		(unit 1)
-		(body_style 1)
-		(exclude_from_sim no)
-		(in_bom yes)
-		(on_board yes)
-		(in_pos_files yes)
-		(dnp no)
-		(property "Reference" "AE1"
-			(at 36.576 87.122 0)
-			(show_name no)
-			(do_not_autoplace no)
-			(effects
-				(font
-					(size 1.27 1.27)
-				)
-			)
-		)
-		(property "Value" "Antenna_Shield"
-			(at 36.576 84.582 0)
-			(show_name no)
-			(do_not_autoplace no)
-			(effects
-				(font
-					(size 1.27 1.27)
-				)
-			)
-		)
-		(property "Footprint" "Footprints:SMA_EdgeMount"
-			(at 36.83 80.01 0)
-			(hide yes)
-			(show_name no)
-			(do_not_autoplace no)
-			(effects
-				(font
-					(size 1.27 1.27)
-				)
-			)
-		)
-		(property "Datasheet" ""
-			(at 36.83 80.01 0)
-			(hide yes)
-			(show_name no)
-			(do_not_autoplace no)
-			(effects
-				(font
-					(size 1.27 1.27)
-				)
-			)
-		)
-		(property "Description" "Antenna with extra pin for shielding"
-			(at 36.83 77.47 0)
-			(hide yes)
-			(show_name no)
-			(do_not_autoplace no)
-			(effects
-				(font
-					(size 1.27 1.27)
-				)
-			)
-		)
-		(pin "2"
-		)
-		(pin "1"
-		)
-		(instances
-			(project "SUITON_mini"
-				(path "/651dea4f-1e55-4052-accd-e9842c395f76/cbc1e4b3-87c3-4a09-a481-980e2b628052"
-					(reference "AE1")
-					(unit 1)
-				)
