File: SUITON_telem/SUITON_mini/pyro.kicad_sch (KiCad schematic)
At the start: 13 parts, among them J5 Conn_01x03_Pin, U12 TPS1H200AQDGNRQ1, U14 TPS1H200AQDGNRQ1

Commit message: New rf module
Parts:
- U12, U14: DESCRIPTION 40-V, 200-mΩ, 1-ch automotive smart high-side switch with a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 -> (none)

Commit message: Shape
Parts:
- J5: footprint (none) -> TerminalBlock_Phoenix:TerminalBlock_Phoenix_MPT-0,5-3-2.54_1x03_P2.54mm_Horizontal
Changed lines of the file:
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@@
 			)
 		)
-		(property "Footprint" ""
+		(property "Footprint" "TerminalBlock_Phoenix:TerminalBlock_Phoenix_MPT-0,5-3-2.54_1x03_P2.54mm_Horizontal"
 			(at 134.62 97.79 0)
 			(hide yes)
